Commit message: Uniformization of topic names between simulation and the robot platform (lasers, odometry, twist).

File: guardian_description/urdf/v7/guardian_tracks_laser_up.urdf (copy).xacro (robot description, xacro)
@@ -1,7 +1,6 @@
 <?xml version="1.0"?>
-<robot name="gball" xmlns:xacro="http://www.ros.org/wiki/xacro">
+<robot name="guardian_tracks" xmlns:xacro="http://www.ros.org/wiki/xacro">
   <!-- Import all Gazebo-customization elements, including Gazebo colors -->
   <xacro:include filename="$(find guardian_description)/urdf/v7/guardian.gazebo" />
-<!--   <xacro:include filename="$(find guardian_description)/urdf/sensors/kinect.urdf.xacro"/> -->
   <!-- Robot mechanical and motor parameters -->
   <xacro:property name="PI" value="3.1415926535897931"/>
@@ -19,4 +18,6 @@
   <xacro:property name="ptz_joint_damping" value="0.1" />
   <xacro:property name="ptz_mechanical_reduction" value="1.0" />
+  <xacro:property name="laser_offset_x" value="-0.048" />
+  <xacro:property name="laser_offset_z" value="0.06" />
   <!-- Used for fixing robot to Gazebo 'base_link' -->
   <!-- link name="world"/>
@@ -46,5 +47,5 @@
       This moves the joint to 0,0,0 where we want it for rviz, etc. -->
      <!-- origin xyz="0 0 0.130" rpy="0 0 0" / -->
-     <origin xyz="0 0 0.18" rpy="0 0 0" />
+     <origin xyz="0 0 0.069" rpy="0 0 0" />
      <parent link="base_footprint"/>
      <child link="base_link" />
@@ -108,9 +109,9 @@
        <origin xyz="0 0 0" rpy="0 0 0" />
        <geometry>
-	 	 <mesh filename="package://guardian_description/meshes/others/v5/trackV5_l.dae"/>
-       </geometry>
-	   <material name="black">
-		 <color rgba="0.1 0.1 0.1 1"/>
-       </material>
+	 <mesh filename="package://guardian_description/meshes/others/v5/trackV5_l.dae"/>
+       </geometry>
+	<material name="black">
+		<color rgba="0.1 0.1 0.1 1"/>
+      	</material>
     </visual>
     <collision>
@@ -127,5 +128,5 @@
   </joint>
   <!-- BACK LEFT WHEEL (GREY) -->
-  <link name="back_left_wheel">
+  <!-- <link name="back_left_wheel">
     <inertial>
       <mass value="4.5" />
@@ -133,19 +134,4 @@
       <inertia  ixx="0.059" ixy="0.0"  ixz="0.0"  iyy="0.055"  iyz="0.0"  izz="0.059" />
     </inertial>
-    <visual>
-       <origin xyz="0 0 0" rpy="0 0 3.1416" />
-       <geometry>
-	 	 <mesh filename="package://guardian_description/meshes/wheel.dae"/>
-       </geometry>
-	   <material name="grey">
-		 <color rgba="0.3 0.3 0.3 1"/>
-       </material>
-    </visual>
-    <collision>
-       <origin xyz="0 0 0" rpy="0 0 3.1416" />
-       <geometry>
-         <mesh filename="package://guardian_description/meshes/wheel.dae"/>
-       </geometry>
-    </collision>
   </link>
   <joint name="joint_back_left_wheel" type="continuous">
@@ -162,10 +148,10 @@
      <actuator name="joint_blw_motor">
 	    <hardwareInterface>EffortJointInterface</hardwareInterface>
-		<!-- hardwareInterface>VelocityJointInterface</hardwareInterface -->
+		hardwareInterface>VelocityJointInterface</hardwareInterface
         <mechanicalReduction>${wheel_mechanical_reduction}</mechanicalReduction>
-     	<!-- motorTorqueConstant>1</motorTorqueConstant -->
+     	motorTorqueConstant>1</motorTorqueConstant
      </actuator>
   </transmission>
-  <!-- BACK RIGHT WHEEL (BLACK) -->
+  BACK RIGHT WHEEL (BLACK)
   <link name="back_right_wheel">
     <inertial>
@@ -174,19 +160,4 @@
       <inertia  ixx="0.059" ixy="0.0"  ixz="0.0"  iyy="0.055"  iyz="0.0"  izz="0.059" />
     </inertial>
-    <visual>
-       <origin xyz="0 0 0" rpy="0 0 0" />
-       <geometry>
-         <mesh filename="package://guardian_description/meshes/wheel.dae"/>
-       </geometry>
-	   <material name="gray">
-		 <color rgba="0.3 0.3 0.3 1"/>
-       </material>
-    </visual>
-    <collision>
-       <origin xyz="0 0 0" rpy="0 0 0" />
-       <geometry>
-         <mesh filename="package://guardian_description/meshes/wheel.dae"/>
-       </geometry>
-    </collision>
   </link>
   <joint name="joint_back_right_wheel" type="continuous">
@@ -203,10 +174,10 @@
     <actuator name="joint_brw_motor">
 	   <hardwareInterface>EffortJointInterface</hardwareInterface>
-       <!-- hardwareInterface>VelocityJointInterface</hardwareInterface -->
+       hardwareInterface>VelocityJointInterface</hardwareInterface
        <mechanicalReduction>${wheel_mechanical_reduction}</mechanicalReduction>
-	   <!-- motorTorqueConstant>1</motorTorqueConstant -->
+	   motorTorqueConstant>1</motorTorqueConstant
     </actuator>
   </transmission>
-  <!-- FRONT LEFT WHEEL (GREY) -->
+  FRONT LEFT WHEEL (GREY)
   <link name="front_left_wheel">
     <inertial>
@@ -215,19 +186,4 @@
       <inertia  ixx="0.059" ixy="0.0"  ixz="0.0"  iyy="0.055"  iyz="0.0"  izz="0.059" />
     </inertial>
-    <visual>
-       <origin xyz="0 0 0" rpy="0 0 3.1416" />
-       <geometry>
-         <mesh filename="package://guardian_description/meshes/wheel.dae"/>
-       </geometry>
-	   <material name="grey">
-		 <color rgba="0.3 0.3 0.3 1"/>
-       </material>
-    </visual>
-    <collision>
-       <origin xyz="0 0 0" rpy="0 0 3.1416" />
-       <geometry>
-         <mesh filename="package://guardian_description/meshes/wheel.dae"/>
-       </geometry>
-    </collision>
   </link>
   <joint name="joint_front_left_wheel" type="continuous">
@@ -244,10 +200,10 @@
      <actuator name="joint_flw_motor">
 	   <hardwareInterface>EffortJointInterface</hardwareInterface>
-       <!-- hardwareInterface>VelocityJointInterface</hardwareInterface -->
+       hardwareInterface>VelocityJointInterface</hardwareInterface
        <mechanicalReduction>${wheel_mechanical_reduction}</mechanicalReduction>
-       <!-- motorTorqueConstant>1</motorTorqueConstant -->
+       motorTorqueConstant>1</motorTorqueConstant
      </actuator>
   </transmission>
-  <!-- FRONT RIGHT WHEEL (GREY) -->
+  FRONT RIGHT WHEEL (GREY)
   <link name="front_right_wheel">
     <inertial>
@@ -256,19 +212,4 @@
       <inertia  ixx="0.059" ixy="0.0"  ixz="0.0"  iyy="0.055"  iyz="0.0"  izz="0.059" />
     </inertial>
-    <visual>
-       <origin xyz="0 0 0" rpy="0 0 0" />
-       <geometry>
-         <mesh filename="package://guardian_description/meshes/wheel.dae"/>
-       </geometry>
-	   <material name="grey">
-		 <color rgba="0.3 0.3 0.3 1"/>
-       </material>
-    </visual>
-    <collision>
-       <origin xyz="0 0 0" rpy="0 0 0" />
-       <geometry>
-         <mesh filename="package://guardian_description/meshes/wheel.dae"/>
-       </geometry>
-    </collision>
   </link>
   <joint name="joint_front_right_wheel" type="continuous">
@@ -285,11 +226,11 @@
      <actuator name="joint_frw_motor">
 	   <hardwareInterface>EffortJointInterface</hardwareInterface>
-	   <!-- hardwareInterface>VelocityJointInterface</hardwareInterface -->
+	   hardwareInterface>VelocityJointInterface</hardwareInterface
        <mechanicalReduction>${wheel_mechanical_reduction}</mechanicalReduction>
-       <!-- motorTorqueConstant>1</motorTorqueConstant -->
+       motorTorqueConstant>1</motorTorqueConstant
      </actuator>
-     <!-- motorTorqueConstant>1</motorTorqueConstant -->
-  </transmission>
-<!-- 	<sensor_kinect  parent="base_link"/> -->
+     motorTorqueConstant>1</motorTorqueConstant
+  </transmission>
+ -->
   <!-- HOKUYO BACK SENSOR -->
   <joint name="hokuyo_back_laser_joint" type="fixed">
@@ -375,5 +316,5 @@
   <joint name="hokuyo_frontal_laser_joint" type="fixed">
      <axis xyz="0 1 0" />
-     <origin xyz="0.066 0 0.0"/>
+     <origin xyz="${laser_offset_x+0.066} 0 ${laser_offset_z}"/>
      <parent link="laser_tilt_link"/>
      <child link="hokuyo_frontal_laser_link"/>

File: guardian_description/urdf/v7/guardian_tracks_laser_up.urdf.xacro (robot description, xacro)
@@ -1,7 +1,6 @@
 <?xml version="1.0"?>
-<robot name="gball" xmlns:xacro="http://www.ros.org/wiki/xacro">
+<robot name="guardian_tracks" xmlns:xacro="http://www.ros.org/wiki/xacro">
   <!-- Import all Gazebo-customization elements, including Gazebo colors -->
   <xacro:include filename="$(find guardian_description)/urdf/v7/guardian.gazebo" />
-<!--   <xacro:include filename="$(find guardian_description)/urdf/sensors/kinect.urdf.xacro"/> -->
   <!-- Robot mechanical and motor parameters -->
   <xacro:property name="PI" value="3.1415926535897931"/>
@@ -19,4 +18,6 @@
   <xacro:property name="ptz_joint_damping" value="0.1" />
   <xacro:property name="ptz_mechanical_reduction" value="1.0" />
+  <xacro:property name="laser_offset_x" value="-0.048" />
+  <xacro:property name="laser_offset_z" value="0.06" />
   <!-- Used for fixing robot to Gazebo 'base_link' -->
   <!-- link name="world"/>
@@ -35,10 +36,10 @@
           </geometry>
       </visual>
-      <collision>
+     <!--  <collision>
           <origin xyz="0 0 0" rpy="0 0 0" />
           <geometry>
             <box size="0.001 0.001 0.001" />
          </geometry>
-     </collision>
+     </collision> -->
   </link>
   <joint name="base_footprint_joint" type="fixed">
@@ -46,5 +47,5 @@
       This moves the joint to 0,0,0 where we want it for rviz, etc. -->
      <!-- origin xyz="0 0 0.130" rpy="0 0 0" / -->
-     <origin xyz="0 0 0.18" rpy="0 0 0" />
+     <origin xyz="0 0 0.069" rpy="0 0 0" />
      <parent link="base_footprint"/>
      <child link="base_link" />
@@ -60,11 +61,14 @@
        <origin xyz="0 0 0" rpy="0 0 0" />
        <geometry>
-	 <mesh filename="package://guardian_description/meshes/chassis/v7/chassisV7.dae"/>
-       </geometry>
+	 		<mesh filename="package://guardian_description/meshes/chassis/v7/chassisV7.stl"/>
+       </geometry>
+       <material name="DarkGrey">
+			<color rgba="0.4 0.4 0.4 1.0" />
+		</material>
     </visual>
     <collision>
        <origin xyz="0 0 0" rpy="0 0 0 " />
        <geometry>
-         <mesh filename="package://guardian_description/meshes/chassis/v7/chassisV7.dae"/>
+         <mesh filename="package://guardian_description/meshes/chassis/v7/chassisV7.stl"/>
        </geometry>
     </collision>
@@ -80,5 +84,5 @@
         <origin xyz="0 0 0" rpy="0 0 0" />
         <geometry>
-	 <mesh filename="package://guardian_description/meshes/others/v5/trackV5_l.dae"/>
+	 <mesh filename="package://guardian_description/meshes/others/v5/trackV5_l.stl"/>
         </geometry>
 	<material name="black">
@@ -89,5 +93,5 @@
        <origin xyz="0 0 0" rpy="0 0 0" />
        <geometry>
-         <mesh filename="package://guardian_description/meshes/others/v5/trackV5_l.dae"/>
+         <mesh filename="package://guardian_description/meshes/others/v5/trackV5_l.stl"/>
        </geometry>
     </collision>
@@ -108,14 +112,14 @@
        <origin xyz="0 0 0" rpy="0 0 0" />
        <geometry>
-	 	 <mesh filename="package://guardian_description/meshes/others/v5/trackV5_l.dae"/>
-       </geometry>
-	   <material name="black">
-		 <color rgba="0.1 0.1 0.1 1"/>
-       </material>
-    </visual>
-    <collision>
-       <origin xyz="0 0 0" rpy="0 0 0" />
-       <geometry>
-         <mesh filename="package://guardian_description/meshes/others/v5/trackV5_l.dae"/>
+	 <mesh filename="package://guardian_description/meshes/others/v5/trackV5_l.stl"/>
+       </geometry>
+	<material name="black">
+		<color rgba="0.1 0.1 0.1 1"/>
+      	</material>
+    </visual>
+    <collision>
+       <origin xyz="0 0 0" rpy="0 0 0" />
+       <geometry>
+         <mesh filename="package://guardian_description/meshes/others/v5/trackV5_l.stl"/>
        </geometry>
     </collision>
@@ -126,170 +130,4 @@
     <origin xyz="0.0 0.0 0.0" rpy="0 0 3.1415926535" />
   </joint>
-  <!-- BACK LEFT WHEEL (GREY) -->
-  <link name="back_left_wheel">
-    <inertial>
-      <mass value="4.5" />
-      <origin xyz="0 0 0" rpy="0 0 3.1416"/>
-      <inertia  ixx="0.059" ixy="0.0"  ixz="0.0"  iyy="0.055"  iyz="0.0"  izz="0.059" />
-    </inertial>
-    <visual>
-       <origin xyz="0 0 0" rpy="0 0 3.1416" />
-       <geometry>
-	 	 <mesh filename="package://guardian_description/meshes/wheel.dae"/>
-       </geometry>
-	   <material name="grey">
-		 <color rgba="0.3 0.3 0.3 1"/>
-       </material>
-    </visual>
-    <collision>
-       <origin xyz="0 0 0" rpy="0 0 3.1416" />
-       <geometry>
-         <mesh filename="package://guardian_description/meshes/wheel.dae"/>
-       </geometry>
-    </collision>
-  </link>
-  <joint name="joint_back_left_wheel" type="continuous">
-    <parent link="base_link"/>
-    <child link="back_left_wheel"/>
-    <origin xyz="-${wheel_offset_x} ${wheel_offset_y} 0" rpy="0 0 0" />
-    <axis xyz="0 1 0" rpy="0 0 0" />
-    <limit effort="${wheel_joint_effort_limit}" velocity="${wheel_joint_velocity_limit}"/>
-    <joint_properties damping="${wheel_joint_damping}" friction="{wheel_joint_friction}"/>
-  </joint>
-  <transmission name="joint_blw_trans">
-	 <type>transmission_interface/SimpleTransmission</type>
-     <joint name="joint_back_left_wheel" />
-     <actuator name="joint_blw_motor">
-	    <hardwareInterface>EffortJointInterface</hardwareInterface>
-		<!-- hardwareInterface>VelocityJointInterface</hardwareInterface -->
-        <mechanicalReduction>${wheel_mechanical_reduction}</mechanicalReduction>
-     	<!-- motorTorqueConstant>1</motorTorqueConstant -->
-     </actuator>
-  </transmission>
-  <!-- BACK RIGHT WHEEL (BLACK) -->
-  <link name="back_right_wheel">
-    <inertial>
-      <mass value="4.5" />
-      <origin xyz="0 0 0" rpy="0 0 0"/>
-      <inertia  ixx="0.059" ixy="0.0"  ixz="0.0"  iyy="0.055"  iyz="0.0"  izz="0.059" />
-    </inertial>
-    <visual>
-       <origin xyz="0 0 0" rpy="0 0 0" />
-       <geometry>
-         <mesh filename="package://guardian_description/meshes/wheel.dae"/>
-       </geometry>
-	   <material name="gray">
-		 <color rgba="0.3 0.3 0.3 1"/>
-       </material>
-    </visual>
-    <collision>
-       <origin xyz="0 0 0" rpy="0 0 0" />
-       <geometry>
-         <mesh filename="package://guardian_description/meshes/wheel.dae"/>
-       </geometry>
-    </collision>
-  </link>
-  <joint name="joint_back_right_wheel" type="continuous">
-    <parent link="base_link"/>
-    <child link="back_right_wheel"/>
-    <origin xyz="-${wheel_offset_x} -${wheel_offset_y} 0" rpy="0 0 0" />
-    <axis xyz="0 1 0" rpy="0 0 0" />
-    <limit effort="${wheel_joint_effort_limit}" velocity="${wheel_joint_velocity_limit}"/>
-    <joint_properties damping="${wheel_joint_damping}" friction="{wheel_joint_friction}"/>
-  </joint>
-  <transmission name="joint_brw_trans">
-    <type>transmission_interface/SimpleTransmission</type>
-    <joint name="joint_back_right_wheel" />
-    <actuator name="joint_brw_motor">
-	   <hardwareInterface>EffortJointInterface</hardwareInterface>
-       <!-- hardwareInterface>VelocityJointInterface</hardwareInterface -->
-       <mechanicalReduction>${wheel_mechanical_reduction}</mechanicalReduction>
-	   <!-- motorTorqueConstant>1</motorTorqueConstant -->
-    </actuator>
-  </transmission>
-  <!-- FRONT LEFT WHEEL (GREY) -->
-  <link name="front_left_wheel">
-    <inertial>
-      <mass value="4.5" />
-      <origin xyz="0 0 0" rpy="0 0 3.1416"/>
-      <inertia  ixx="0.059" ixy="0.0"  ixz="0.0"  iyy="0.055"  iyz="0.0"  izz="0.059" />
-    </inertial>
-    <visual>
-       <origin xyz="0 0 0" rpy="0 0 3.1416" />
-       <geometry>
-         <mesh filename="package://guardian_description/meshes/wheel.dae"/>
-       </geometry>
-	   <material name="grey">
-		 <color rgba="0.3 0.3 0.3 1"/>
-       </material>
-    </visual>
-    <collision>
-       <origin xyz="0 0 0" rpy="0 0 3.1416" />
-       <geometry>
-         <mesh filename="package://guardian_description/meshes/wheel.dae"/>
-       </geometry>
-    </collision>
-  </link>
-  <joint name="joint_front_left_wheel" type="continuous">
-    <parent link="base_link"/>
-    <child link="front_left_wheel"/>
-    <origin xyz="${wheel_offset_x} ${wheel_offset_y} 0" rpy="0 0 0" />
-    <axis xyz="0 1 0" rpy="0 0 0" />
-    <limit effort="${wheel_joint_effort_limit}" velocity="${wheel_joint_velocity_limit}"/>
-    <joint_properties damping="${wheel_joint_damping}" friction="{wheel_joint_friction}"/>
-  </joint>
-  <transmission name="joint_flw_trans">
-	 <type>transmission_interface/SimpleTransmission</type>
-     <joint name="joint_front_left_wheel" />
-     <actuator name="joint_flw_motor">
-	   <hardwareInterface>EffortJointInterface</hardwareInterface>
-       <!-- hardwareInterface>VelocityJointInterface</hardwareInterface -->
-       <mechanicalReduction>${wheel_mechanical_reduction}</mechanicalReduction>
-       <!-- motorTorqueConstant>1</motorTorqueConstant -->
-     </actuator>
-  </transmission>
-  <!-- FRONT RIGHT WHEEL (GREY) -->
-  <link name="front_right_wheel">
-    <inertial>
-      <mass value="4.5" />
-      <origin xyz="0 0 0" rpy="0 0 0"/>
-      <inertia  ixx="0.059" ixy="0.0"  ixz="0.0"  iyy="0.055"  iyz="0.0"  izz="0.059" />
-    </inertial>
-    <visual>
-       <origin xyz="0 0 0" rpy="0 0 0" />
-       <geometry>
-         <mesh filename="package://guardian_description/meshes/wheel.dae"/>
-       </geometry>
-	   <material name="grey">
-		 <color rgba="0.3 0.3 0.3 1"/>
-       </material>
-    </visual>
-    <collision>
-       <origin xyz="0 0 0" rpy="0 0 0" />
-       <geometry>
-         <mesh filename="package://guardian_description/meshes/wheel.dae"/>
-       </geometry>
-    </collision>
-  </link>
-  <joint name="joint_front_right_wheel" type="continuous">
-    <parent link="base_link"/>
-    <child link="front_right_wheel"/>
-    <origin xyz="${wheel_offset_x} -${wheel_offset_y} 0" rpy="0 0 0" />
-    <axis xyz="0 1 0" rpy="0 0 0" />
-    <limit effort="${wheel_joint_effort_limit}" velocity="${wheel_joint_velocity_limit}"/>
-    <joint_properties damping="${wheel_joint_damping}" friction="{wheel_joint_friction}"/>
-  </joint>
-  <transmission name="joint_frw_trans">
-	 <type>transmission_interface/SimpleTransmission</type>
-     <joint name="joint_front_right_wheel" />
-     <actuator name="joint_frw_motor">
-	   <hardwareInterface>EffortJointInterface</hardwareInterface>
-	   <!-- hardwareInterface>VelocityJointInterface</hardwareInterface -->
-       <mechanicalReduction>${wheel_mechanical_reduction}</mechanicalReduction>
-       <!-- motorTorqueConstant>1</motorTorqueConstant -->
-     </actuator>
-     <!-- motorTorqueConstant>1</motorTorqueConstant -->
-  </transmission>
-<!-- 	<sensor_kinect  parent="base_link"/> -->
   <!-- HOKUYO BACK SENSOR -->
   <joint name="hokuyo_back_laser_joint" type="fixed">
@@ -375,5 +213,5 @@
   <joint name="hokuyo_frontal_laser_joint" type="fixed">
      <axis xyz="0 1 0" />
-     <origin xyz="0.066 0 0.0"/>
+     <origin xyz="${laser_offset_x+0.066} 0 ${laser_offset_z}"/>
      <parent link="laser_tilt_link"/>
      <child link="hokuyo_frontal_laser_link"/>
