Commit message: Uniformization of topic names between simulation and the robot platform (lasers, odometry, twist).

File: guardian_description/urdf/v7/guardian_wheels_laser_up.urdf.xacro (robot description, xacro)
@@ -3,5 +3,5 @@
   <!-- Import all Gazebo-customization elements, including Gazebo colors -->
   <xacro:include filename="$(find guardian_description)/urdf/v7/guardian.gazebo" />
-<!--   <xacro:include filename="$(find guardian_description)/urdf/sensors/kinect.urdf.xacro"/> -->
+  <xacro:include filename="$(find guardian_description)/urdf/sensors/kinect.urdf.xacro"/>
   <!-- Robot mechanical and motor parameters -->
   <xacro:property name="PI" value="3.1415926535897931"/>
@@ -19,4 +19,10 @@
   <xacro:property name="ptz_joint_damping" value="0.1" />
   <xacro:property name="ptz_mechanical_reduction" value="1.0" />
+   <xacro:property name="laser_offset_x" value="-0.048" />
+  <xacro:property name="laser_offset_z" value="0.06" />
+  <xacro:property name="simple_wheel_length" value="0.115" />
+  <xacro:property name="simple_wheel_radius" value="0.185" />
+  <xacro:property name="wheel_origin_y" value="0.0415" />
+  <xacro:property name="wheel_offset_y_a" value="0.306" />
   <!-- Used for fixing robot to Gazebo 'base_link' -->
   <!-- link name="world"/>
@@ -35,10 +41,10 @@
           </geometry>
       </visual>
-      <collision>
+     <!--  <collision>
           <origin xyz="0 0 0" rpy="0 0 0" />
           <geometry>
             <box size="0.001 0.001 0.001" />
          </geometry>
-     </collision>
+     </collision> -->
   </link>
   <joint name="base_footprint_joint" type="fixed">
@@ -50,8 +56,8 @@
      <child link="base_link" />
   </joint>
-  <!-- BASE_LINK (RED) -->
+  <!-- BASE_LINK (DarkGrey) -->
   <link name="base_link">
     <inertial>
-      <mass value="95.0" />
+      <mass value="33.50" /> <!-- 95.0 -->
       <origin xyz="0 0 0" />
       <inertia  ixx="3.737" ixy="0.008"  ixz="-0.144"  iyy="8.311"  iyz="-0.004"  izz="8.893" />
@@ -60,16 +66,20 @@
        <origin xyz="0 0 0" rpy="0 0 0" />
        <geometry>
-	 <mesh filename="package://guardian_description/meshes/chassis/v7/chassisV7.dae"/>
-       </geometry>
-    </visual>
-    <collision>
-       <origin xyz="0 0 0" rpy="0 0 0 " />
-       <geometry>
-         <mesh filename="package://guardian_description/meshes/chassis/v7/chassisV7.dae"/>
-       </geometry>
-    </collision>
-  </link>
-  <!-- LEFT TRACK (BLACK) -->
-  <link name="left_track">
+	 <mesh filename="package://guardian_description/meshes/chassis/v7/chassisV7.stl"/>
+       </geometry>
+		<material name="DarkGrey">
+			<color rgba="0.4 0.4 0.4 1.0" />
+		</material>
+    </visual>
+    <collision>
+       <origin xyz="0 0 0.08" rpy="0 0 0 " />
+       <geometry>
+         <mesh filename="package://guardian_description/meshes/chassis/v7/chassisV7.stl"/>
+       </geometry>
+    </collision>
+  </link>
+<!-- ################# TRACKS ################# -->
+  <!-- RIGHT TRACK (BLACK) -->
+  <link name="right_track">
     <inertial>
       <mass value="1.250" />
@@ -78,26 +88,26 @@
     </inertial>
     <visual>
-        <origin xyz="0 0 0" rpy="0 0 0" />
-        <geometry>
-	 <mesh filename="package://guardian_description/meshes/others/v5/trackV5_l.dae"/>
-        </geometry>
-	<material name="black">
-  		<color rgba="0.1 0.1 0.1 1"/>
-      	</material>
-    </visual>
-    <collision>
-       <origin xyz="0 0 0" rpy="0 0 0" />
-       <geometry>
-         <mesh filename="package://guardian_description/meshes/others/v5/trackV5_l.dae"/>
-       </geometry>
-    </collision>
-  </link>
-  <joint name="joint_left_track" type="fixed">
-    <parent link="base_link"/>
-    <child link="left_track"/>
+      <origin xyz="0 0 0" rpy="0 0 0" />
+      <geometry>
+	 	 <mesh filename="package://guardian_description/meshes/others/v5/trackV5_l.stl"/>
+      </geometry>
+	  <material name="black">
+  		 <color rgba="0.1 0.1 0.1 1"/>
+      </material>
+    </visual>
+    <collision>
+       <origin xyz="0 0 0" rpy="0 0 0" />
+       <geometry>
+         <mesh filename="package://guardian_description/meshes/others/v5/trackV5_l.stl"/>
+       </geometry>
+    </collision>
+  </link>
+  <joint name="joint_right_track" type="fixed">
+    <parent link="base_link"/>
+    <child link="right_track"/>
     <origin xyz="0.0 0.0 0.0" rpy="0 0 0" />
   </joint>
-  <!-- RIGHT TRACK (BLACK) -->
-  <link name="right_track">
+  <!-- LEFT TRACK (BLACK) -->
+  <link name="left_track">
     <inertial>
       <mass value="1.250" />
@@ -108,5 +118,5 @@
        <origin xyz="0 0 0" rpy="0 0 0" />
        <geometry>
-	 	 <mesh filename="package://guardian_description/meshes/others/v5/trackV5_l.dae"/>
+	 	  <mesh filename="package://guardian_description/meshes/others/v5/trackV5_l.stl"/>
        </geometry>
 	   <material name="black">
@@ -117,33 +127,34 @@
        <origin xyz="0 0 0" rpy="0 0 0" />
        <geometry>
-         <mesh filename="package://guardian_description/meshes/others/v5/trackV5_l.dae"/>
-       </geometry>
-    </collision>
-  </link>
-  <joint name="joint_right_track" type="fixed">
-    <parent link="base_link"/>
-    <child link="right_track"/>
+         <mesh filename="package://guardian_description/meshes/others/v5/trackV5_l.stl"/>
+       </geometry>
+    </collision>
+  </link>
+  <joint name="joint_left_track" type="fixed">
+    <parent link="base_link"/>
+    <child link="left_track"/>
     <origin xyz="0.0 0.0 0.0" rpy="0 0 3.1415926535" />
   </joint>
+<!-- ################# WHEELS ################# -->
   <!-- BACK LEFT WHEEL (GREY) -->
   <link name="back_left_wheel">
     <inertial>
       <mass value="4.5" />
-      <origin xyz="0 0 0" rpy="0 0 3.1416"/>
+      <origin xyz="0 0 0" rpy="0 0 ${PI}"/>
       <inertia  ixx="0.059" ixy="0.0"  ixz="0.0"  iyy="0.055"  iyz="0.0"  izz="0.059" />
     </inertial>
     <visual>
-       <origin xyz="0 0 0" rpy="0 0 3.1416" />
-       <geometry>
-	 	 <mesh filename="package://guardian_description/meshes/wheel.dae"/>
-       </geometry>
-	   <material name="grey">
-		 <color rgba="0.3 0.3 0.3 1"/>
+       <origin xyz="0 0 0" rpy="0 0 ${PI}" />
+       <geometry>
+	 	  <mesh filename="package://guardian_description/meshes/wheel.stl"/>
+       </geometry>
+	   <material name="black">
+		  <color rgba="0.1 0.1 0.1 1"/>
        </material>
     </visual>
     <collision>
-       <origin xyz="0 0 0" rpy="0 0 3.1416" />
-       <geometry>
-         <mesh filename="package://guardian_description/meshes/wheel.dae"/>
+       <origin xyz="0 0 0" rpy="0 0 ${PI}" />
+       <geometry>
+         <mesh filename="package://guardian_description/meshes/wheel.stl"/>
        </geometry>
     </collision>
@@ -152,5 +163,5 @@
     <parent link="base_link"/>
     <child link="back_left_wheel"/>
-    <origin xyz="-${wheel_offset_x} ${wheel_offset_y} 0" rpy="0 0 0" />
+    <origin xyz="-${wheel_offset_x} -${wheel_offset_y} 0" rpy="0 0 0" />
     <axis xyz="0 1 0" rpy="0 0 0" />
     <limit effort="${wheel_joint_effort_limit}" velocity="${wheel_joint_velocity_limit}"/>
@@ -177,5 +188,5 @@
        <origin xyz="0 0 0" rpy="0 0 0" />
        <geometry>
-         <mesh filename="package://guardian_description/meshes/wheel.dae"/>
+         <mesh filename="package://guardian_description/meshes/wheel.stl"/>
        </geometry>
 	   <material name="gray">
@@ -193,5 +204,5 @@
     <parent link="base_link"/>
     <child link="back_right_wheel"/>
-    <origin xyz="-${wheel_offset_x} -${wheel_offset_y} 0" rpy="0 0 0" />
+    <origin xyz="-${wheel_offset_x} ${wheel_offset_y} 0" rpy="0 0 0" />
     <axis xyz="0 1 0" rpy="0 0 0" />
     <limit effort="${wheel_joint_effort_limit}" velocity="${wheel_joint_velocity_limit}"/>
@@ -216,7 +227,7 @@
     </inertial>
     <visual>
-       <origin xyz="0 0 0" rpy="0 0 3.1416" />
-       <geometry>
-         <mesh filename="package://guardian_description/meshes/wheel.dae"/>
+       <origin xyz="0 -${wheel_origin_y} 0" rpy="0 0 ${PI}" />
+       <geometry>
+         <mesh filename="package://guardian_description/meshes/wheel.stl"/>
        </geometry>
 	   <material name="grey">
@@ -234,5 +245,5 @@
     <parent link="base_link"/>
     <child link="front_left_wheel"/>
-    <origin xyz="${wheel_offset_x} ${wheel_offset_y} 0" rpy="0 0 0" />
+    <origin xyz="${wheel_offset_x} -${wheel_offset_y} 0" rpy="0 0 0" />
     <axis xyz="0 1 0" rpy="0 0 0" />
     <limit effort="${wheel_joint_effort_limit}" velocity="${wheel_joint_velocity_limit}"/>
@@ -259,5 +270,5 @@
        <origin xyz="0 0 0" rpy="0 0 0" />
        <geometry>
-         <mesh filename="package://guardian_description/meshes/wheel.dae"/>
+         <mesh filename="package://guardian_description/meshes/wheel.stl"/>
        </geometry>
 	   <material name="grey">
@@ -268,5 +279,5 @@
        <origin xyz="0 0 0" rpy="0 0 0" />
        <geometry>
-         <mesh filename="package://guardian_description/meshes/wheel.dae"/>
+         <mesh filename="package://guardian_description/meshes/wheel.stl"/>
        </geometry>
     </collision>
@@ -275,5 +286,5 @@
     <parent link="base_link"/>
     <child link="front_right_wheel"/>
-    <origin xyz="${wheel_offset_x} -${wheel_offset_y} 0" rpy="0 0 0" />
+    <origin xyz="${wheel_offset_x} ${wheel_offset_y} 0" rpy="0 0 0" />
     <axis xyz="0 1 0" rpy="0 0 0" />
     <limit effort="${wheel_joint_effort_limit}" velocity="${wheel_joint_velocity_limit}"/>
@@ -291,5 +302,6 @@
      <!-- motorTorqueConstant>1</motorTorqueConstant -->
   </transmission>
-<!-- 	<sensor_kinect  parent="base_link"/> -->
+<!-- ################# SENSORS ################# -->
+  <!--<sensor_kinect  parent="base_link"/>-->
   <!-- HOKUYO BACK SENSOR -->
   <joint name="hokuyo_back_laser_joint" type="fixed">
@@ -375,5 +387,6 @@
   <joint name="hokuyo_frontal_laser_joint" type="fixed">
      <axis xyz="0 1 0" />
-     <origin xyz="0.066 0 0.0"/>
+     <!--<origin xyz="0.066 0 0.0"/> -->
+     <origin xyz="${laser_offset_x+0.066} 0 ${laser_offset_z}"/>
      <parent link="laser_tilt_link"/>
      <child link="hokuyo_frontal_laser_link"/>
@@ -387,10 +400,10 @@
       </geometry>
     </collision>
-    <!-- visual>
+    <visual>
       <origin xyz="0 0 0" rpy="0 0 0"/>
       <geometry>
         <mesh filename="package://guardian_description/meshes/hokuyo-utm30-lx.dae"/>
       </geometry>
-    </visual -->
+    </visual>
     <inertial>
       <mass value="1e-5" />
